Commit message: Sim v0

File: urdf/vehicle_v1_double.xacro (robot description, xacro)
@@ -4,5 +4,5 @@
     <xacro:property name="base_w" value="0.15" />
     <xacro:property name="base_h" value="0.05" />
-    <xacro:property name="wh_l" value="0.02" />
+    <xacro:property name="wh_l" value="0.03" />
     <xacro:property name="wh_r" value="0.025" />
     <xacro:property name="wh_base_l" value="0.26" />
@@ -65,6 +65,6 @@
             <parent link="${name}_j_link" />
             <axis rpy="0 0 0" xyz="0 1 0" />
-            <limit effort="10000" velocity="1000" />
-            <!-- <joint_properties damping="100000" friction="0" /> -->
+            <limit effort="10000" velocity="1" />
+            <!-- <joint_properties damping="10000" friction="0" /> -->
         </joint>
         <joint name="${name}_rev_joint" type="revolute">
@@ -73,10 +73,10 @@
             <parent link="base_link" />
             <axis rpy="0 0 0" xyz="0 0 1" />
-            <limit effort="10000" velocity="1000" lower="-2" upper="2" />
-            <!-- <joint_properties damping="0" friction="0"/> -->
+            <limit effort="10000" velocity="1" lower="-1.57" upper="1.57" />
+            <!-- <joint_properties damping="10000" friction="0"/> -->
         </joint>
         <link name="${name}_wheel_link">
             <inertial>
-                <mass value="0.001" />
+                <mass value="0.2" />
                 <origin rpy="0 1.5707 1.5707" xyz="0 0 0" />
                 <inertia ixx="0.000526666666667" ixy="0" ixz="0" iyy="0.000526666666667" iyz="0" izz="0.001" />
@@ -87,14 +87,4 @@
                     <cylinder length="${wh_l}" radius="${wh_r}" />
                 </geometry>
-                <!-- <surface>
-                    <friction>
-                      <ode>
-                        <mu>0.1</mu>
-                        <mu2>0.1</mu2>
-                        <slip1>1.0</slip1>
-                        <slip2>1.0</slip2>
-                      </ode>
-                    </friction>
-                  </surface> -->
             </collision>
             <visual>
@@ -115,8 +105,8 @@
             <type>transmission_interface/SimpleTransmission</type>
             <joint name="${name}_rev_joint">
-                <hardwareInterface>PositionJointInterface</hardwareInterface>
+                <hardwareInterface>EffortJointInterface</hardwareInterface>
             </joint>
             <actuator name="${name}_rev_motor">
-                <hardwareInterface>PositionJointInterface</hardwareInterface>
+                <hardwareInterface>EffortJointInterface</hardwareInterface>
                 <mechanicalReduction>1</mechanicalReduction>
             </actuator>
@@ -125,17 +115,82 @@
             <type>transmission_interface/SimpleTransmission</type>
             <joint name="${name}_cont_joint">
-                <hardwareInterface>VelocityJointInterface</hardwareInterface>
+                <hardwareInterface>EffortJointInterface</hardwareInterface>
             </joint>
             <actuator name="${name}_cont_motor">
-                <hardwareInterface>VelocityJointInterface</hardwareInterface>
+                <hardwareInterface>EffortJointInterface</hardwareInterface>
                 <mechanicalReduction>1</mechanicalReduction>
             </actuator>
         </transmission>
     </xacro:macro>
-    <xacro:wheel name="back" xyz="${-wh_base_l/2} ${0} ${wh_base_z}" />
-    <xacro:wheel name="front" xyz="${wh_base_l/2} ${0} ${wh_base_z}" />
-    <!-- <xacro:wheel name="front_left" xyz="${wh_base_l/2} ${wh_base_w/2} ${wh_base_z}" />
+    <xacro:macro name="wheel_b" params="name xyz">
+        <joint name="${name}_cont_joint" type="continuous">
+            <origin rpy="0 0 0" xyz="0 0 0" />
+            <child link="${name}_wheel_link" />
+            <parent link="${name}_j_link" />
+            <axis rpy="0 0 0" xyz="0 1 0" />
+            <limit effort="10000" velocity="1" />
+            <!-- <joint_properties damping="10000" friction="0" /> -->
+        </joint>
+        <joint name="${name}_f_joint" type="fixed">
+            <origin rpy="0 0 0" xyz="${xyz}" />
+            <child link="${name}_j_link" />
+            <parent link="base_link" />
+            <axis rpy="0 0 0" xyz="0 0 1" />
+                <!-- <limit effort="10000" velocity="1" lower="-1.57" upper="1.57" /> -->
+            <!-- <joint_properties damping="10000" friction="0"/> -->
+        </joint>
+        <link name="${name}_wheel_link">
+            <inertial>
+                <mass value="0.2" />
+                <origin rpy="0 1.5707 1.5707" xyz="0 0 0" />
+                <inertia ixx="0.000526666666667" ixy="0" ixz="0" iyy="0.000526666666667" iyz="0" izz="0.001" />
+            </inertial>
+            <collision>
+                <origin rpy="0 1.5707 1.5707" xyz="0 0 0" />
+                <geometry>
+                    <cylinder length="${wh_l}" radius="${wh_r}" />
+                </geometry>
+            </collision>
+            <visual>
+                <origin rpy="0 1.5707 1.5707" xyz="0 0 0" />
+                <geometry>
+                    <cylinder length="${wh_l}" radius="${wh_r}" />
+                </geometry>
+            </visual>
+        </link>
+        <link name="${name}_j_link">
+            <inertial>
+                <mass value="1e-5" />
+                <origin xyz="0 0 0" rpy="0 0 0" />
+                <inertia ixx="1e-6" ixy="0" ixz="0" iyy="1e-6" iyz="0" izz="1e-6" />
+            </inertial>
+        </link>
+        <!--
+        <transmission name="${name}_rev_trans">
+            <type>transmission_interface/SimpleTransmission</type>
+            <joint name="${name}_rev_joint">
+                <hardwareInterface>EffortJointInterface</hardwareInterface>
+            </joint>
+            <actuator name="${name}_rev_motor">
+                <hardwareInterface>EffortJointInterface</hardwareInterface>
+                <mechanicalReduction>1</mechanicalReduction>
+            </actuator>
+        </transmission>
+        <transmission name="${name}_cont_trans">
+            <type>transmission_interface/SimpleTransmission</type>
+            <joint name="${name}_cont_joint">
+                <hardwareInterface>EffortJointInterface</hardwareInterface>
+            </joint>
+            <actuator name="${name}_cont_motor">
+                <hardwareInterface>EffortJointInterface</hardwareInterface>
+                <mechanicalReduction>1</mechanicalReduction>
+            </actuator>
+            </transmission>
+        -->
+    </xacro:macro>
+    <xacro:wheel_b name="back_left" xyz="${-wh_base_l/2} ${wh_base_w/2} ${wh_base_z}" />
+    <xacro:wheel_b name="back_right" xyz="${-wh_base_l/2} ${-wh_base_w/2} ${wh_base_z}" />
+    <xacro:wheel name="front_left" xyz="${wh_base_l/2} ${wh_base_w/2} ${wh_base_z}" />
     <xacro:wheel name="front_right" xyz="${wh_base_l/2} ${-wh_base_w/2} ${wh_base_z}" />
- -->
     <gazebo reference="camera1_link">
         <sensor type="camera" name="camera1">

Commit message: Sim final

File: urdf/vehicle_v1_double.xacro (robot description, xacro)
@@ -1,17 +1,17 @@
 <?xml version="1.0"?>
 <robot name="vehicle_v1" xmlns:xacro="http://www.ros.org/wiki/xacro">
-    <xacro:property name="base_l" value="0.3" />
-    <xacro:property name="base_w" value="0.15" />
+    <xacro:property name="base_l" value="0.15" />
+    <xacro:property name="base_w" value="0.12" />
     <xacro:property name="base_h" value="0.05" />
-    <xacro:property name="wh_l" value="0.03" />
-    <xacro:property name="wh_r" value="0.025" />
-    <xacro:property name="wh_base_l" value="0.26" />
-    <xacro:property name="wh_base_w" value="0.1" />
-    <xacro:property name="wh_base_z" value="-0.05" />
+    <xacro:property name="wh_l" value="0.033" />
+    <xacro:property name="wh_r" value="0.033" />
+    <xacro:property name="wh_base_l" value="0.162" />
+    <xacro:property name="wh_base_w" value="0.15" />
+    <xacro:property name="wh_base_z" value="0.00" />
     <link name="base_link">
         <!-- pose and inertial -->
         <pose>0 0 0 0 0 0</pose>
         <inertial>
-            <mass value="0.5" />
+            <mass value="2" />
             <origin rpy="0 0 0" xyz="0 0 ${-base_h/2}" />
             <inertia ixx="0.206208333333" ixy="0" ixz="0" iyy="0.206208333333" iyz="0" izz="0.206208333333" />
@@ -34,5 +34,5 @@
     <joint name="camera_joint" type="fixed">
         <axis xyz="0 1 0" />
-        <origin xyz="0.1 0.0 0.2" rpy="0 0.5 0" />
+        <origin xyz="0.121 0.0 0.2" rpy="0 0.68 0" />
         <parent link="base_link" />
         <child link="camera1_link" />
@@ -65,6 +65,7 @@
             <parent link="${name}_j_link" />
             <axis rpy="0 0 0" xyz="0 1 0" />
-            <limit effort="10000" velocity="1" />
-            <!-- <joint_properties damping="10000" friction="0" /> -->
+            <limit effort="10000" velocity="2" />
+            <!-- <joint_properties damping="0" friction="0" /> -->
+            <dynamics damping="0.0" friction="0.0"/>
         </joint>
         <joint name="${name}_rev_joint" type="revolute">
@@ -75,8 +76,10 @@
             <limit effort="10000" velocity="1" lower="-1.57" upper="1.57" />
             <!-- <joint_properties damping="10000" friction="0"/> -->
+            <!-- <joint_properties damping="0" friction="0" /> -->
+            <dynamics damping="0.0" friction="0.0"/>
         </joint>
         <link name="${name}_wheel_link">
             <inertial>
-                <mass value="0.2" />
+                <mass value="0.1" />
                 <origin rpy="0 1.5707 1.5707" xyz="0 0 0" />
                 <inertia ixx="0.000526666666667" ixy="0" ixz="0" iyy="0.000526666666667" iyz="0" izz="0.001" />
@@ -97,7 +100,7 @@
         <link name="${name}_j_link">
             <inertial>
-                <mass value="1e-5" />
+                <mass value="0.1" />
                 <origin xyz="0 0 0" rpy="0 0 0" />
-                <inertia ixx="1e-6" ixy="0" ixz="0" iyy="1e-6" iyz="0" izz="1e-6" />
+                <inertia ixx="1e-3" ixy="0" ixz="0" iyy="1e-3" iyz="0" izz="1e-3" />
             </inertial>
         </link>
@@ -131,4 +134,6 @@
             <limit effort="10000" velocity="1" />
             <!-- <joint_properties damping="10000" friction="0" /> -->
+            <!-- <joint_properties damping="0" friction="0" /> -->
+            <dynamics damping="0.0" friction="0.0"/>
         </joint>
         <joint name="${name}_f_joint" type="fixed">
@@ -139,8 +144,10 @@
                 <!-- <limit effort="10000" velocity="1" lower="-1.57" upper="1.57" /> -->
             <!-- <joint_properties damping="10000" friction="0"/> -->
+            <!-- <joint_properties damping="0" friction="0" /> -->
+            <dynamics damping="0.0" friction="0.0"/>
         </joint>
         <link name="${name}_wheel_link">
             <inertial>
-                <mass value="0.2" />
+                <mass value="0.1" />
                 <origin rpy="0 1.5707 1.5707" xyz="0 0 0" />
                 <inertia ixx="0.000526666666667" ixy="0" ixz="0" iyy="0.000526666666667" iyz="0" izz="0.001" />
@@ -197,8 +204,8 @@
             <update_rate>30.0</update_rate>
             <camera name="head">
-                <horizontal_fov>1.2262634</horizontal_fov>
+                <horizontal_fov>1.5</horizontal_fov>
                 <image>
-                    <width>640</width>
-                    <height>480</height>
+                    <width>800</width>
+                    <height>450</height>
                     <format>R8G8B8</format>
                 </image>

Commit message: Sim final

File: urdf/vehicle_v1_double.xacro (robot description, xacro)
@@ -34,5 +34,5 @@
     <joint name="camera_joint" type="fixed">
         <axis xyz="0 1 0" />
-        <origin xyz="0.121 0.0 0.2" rpy="0 0.68 0" />
+        <origin xyz="0.121 0.0 0.2" rpy="0 0.5 0" />
         <parent link="base_link" />
         <child link="camera1_link" />
@@ -65,6 +65,6 @@
             <parent link="${name}_j_link" />
             <axis rpy="0 0 0" xyz="0 1 0" />
-            <limit effort="10000" velocity="2" />
-            <!-- <joint_properties damping="0" friction="0" /> -->
+            <!-- <limit effort="10000" velocity="2" /> -->
+            <joint_properties damping="0.0" friction="0.0" />
             <dynamics damping="0.0" friction="0.0"/>
         </joint>
@@ -132,5 +132,6 @@
             <parent link="${name}_j_link" />
             <axis rpy="0 0 0" xyz="0 1 0" />
-            <limit effort="10000" velocity="1" />
+            <joint_properties damping="0.0" friction="0.0" />
+            <!-- <limit effort="10000" velocity="2" /> -->
             <!-- <joint_properties damping="10000" friction="0" /> -->
             <!-- <joint_properties damping="0" friction="0" /> -->
@@ -206,6 +207,6 @@
                 <horizontal_fov>1.5</horizontal_fov>
                 <image>
-                    <width>800</width>
-                    <height>450</height>
+                    <width>1280</width>
+                    <height>720</height>
                     <format>R8G8B8</format>
                 </image>
